Commit message: Turn off the d435 camera

File: ugv_gazebo_sim/scout/scout_description/urdf/scout_mini.xacro (robot description, xacro)
@@ -8,11 +8,11 @@
     <xacro:include filename="$(find scout_description)/urdf/scout_mini_wheel_4.xacro" />
     <!-- Variables -->
-    <xacro:property name="M_PI" value="3.14159"/>
+    <xacro:property name="M_PI" value="3.14159" />
     <!-- Vehicle Geometries -->
     <xacro:property name="base_x_size" value="0.6200000" />
     <xacro:property name="base_y_size" value="0.585000" />
     <xacro:property name="base_z_size" value="0.235000" />
-    <xacro:property name="wheelbase" value="0.463951"/>
-    <xacro:property name="track" value="0.416503"/>
+    <xacro:property name="wheelbase" value="0.463951" />
+    <xacro:property name="track" value="0.416503" />
     <xacro:property name="wheel_vertical_offset" value="-0.100998" />
     <xacro:property name="wheel_length" value="0.8e-01" />
@@ -22,5 +22,5 @@
         <origin xyz="0 0 0" rpy="0 0 0" />
     </link>
-     <joint name="base_footprint_joint" type="fixed">
+    <joint name="base_footprint_joint" type="fixed">
         <origin xyz="0 0 ${-wheel_vertical_offset + wheel_radius / 2}" rpy="0 0 0" />
         <parent link="base_footprint" />
@@ -31,6 +31,6 @@
         <visual>
             <origin
-                    xyz="0 0 0.0"
-                    rpy="1.57 0 1.57" />
+                xyz="0 0 0.0"
+                rpy="1.57 0 1.57" />
             <geometry>
                 <mesh filename="package://scout_description/meshes/scout_mini_base_link2.dae" />
@@ -39,10 +39,10 @@
         <collision>
             <origin
-                    xyz="0 0 0"
-                    rpy="1.57 0 1.57" />
-          <geometry>
-            <mesh
-              filename="package://scout_description/meshes/scout_mini_base_link2.dae" />
-          </geometry>
+                xyz="0 0 0"
+                rpy="1.57 0 1.57" />
+            <geometry>
+                <mesh
+                    filename="package://scout_description/meshes/scout_mini_base_link2.dae" />
+            </geometry>
         </collision>
     </link>
@@ -68,5 +68,5 @@
     <!-- motor 1 and 2 (left side) are mechanically installed in a reversed direction -->
     <xacro:scout_mini_wheel_1 wheel_prefix="front_left">
-    <!--<origin
+        <!--<origin
             xyz="0 0 0"
             rpy="0 0 0" />-->
@@ -74,5 +74,5 @@
     </xacro:scout_mini_wheel_1>
     <xacro:scout_mini_wheel_2 wheel_prefix="rear_left">
-    <!--<origin
+        <!--<origin
             xyz="0 0 0"
             rpy="0 0 0" />-->
@@ -80,5 +80,5 @@
     </xacro:scout_mini_wheel_2>
     <xacro:scout_mini_wheel_3 wheel_prefix="front_right">
-    <!--<origin
+        <!--<origin
             xyz="0 0 0"
             rpy="0 0 0" />-->
@@ -86,5 +86,5 @@
     </xacro:scout_mini_wheel_3>
     <xacro:scout_mini_wheel_4 wheel_prefix="rear_right">
-    <!--<origin
+        <!--<origin
            xyz="0 0 0"
            rpy="0 0 0" />-->
@@ -96,55 +96,55 @@
     <joint name="hokuyo_joint" type="fixed">
         <axis xyz="0 1 0" />
-        <origin xyz="0 0 0.14" rpy="0 0 0"/>
-        <parent link="base_link"/>
-        <child link="hokuyo_link"/>
+        <origin xyz="0 0 0.14" rpy="0 0 0" />
+        <parent link="base_link" />
+        <child link="hokuyo_link" />
     </joint>
     <link name="hokuyo_link">
         <collision>
-        <origin xyz="0 0 0" rpy="0 0 0"/>
-        <geometry>
-        <box size="0.1 0.1 0.1"/>
-        </geometry>
+            <origin xyz="0 0 0" rpy="0 0 0" />
+            <geometry>
+                <box size="0.1 0.1 0.1" />
+            </geometry>
         </collision>
         <visual>
-        <origin xyz="0 0 0" rpy="0 0 0"/>
-        <geometry>
-            <mesh filename="package://scout_description/meshes/hokuyo.dae"/>
-        </geometry>
+            <origin xyz="0 0 0" rpy="0 0 0" />
+            <geometry>
+                <mesh filename="package://scout_description/meshes/hokuyo.dae" />
+            </geometry>
         </visual>
         <inertial>
-        <mass value="1e-5" />
-        <origin xyz="0 0 0" rpy="0 0 0"/>
-        <inertia ixx="1e-6" ixy="0" ixz="0" iyy="1e-6" iyz="0" izz="1e-6" />
+            <mass value="1e-5" />
+            <origin xyz="0 0 0" rpy="0 0 0" />
+            <inertia ixx="1e-6" ixy="0" ixz="0" iyy="1e-6" iyz="0" izz="1e-6" />
         </inertial>
     </link>
     <!-- realsense camera -->
-    <xacro:include filename="$(find scout_description)/urdf/_d435.urdf.xacro" />
+    <!-- <xacro:include filename="$(find scout_description)/urdf/_d435.urdf.xacro" />
     <xacro:sensor_d435 parent="base_link" name="camera" topics_ns="camera" publish_pointcloud="true" >
         <origin xyz="0.1 0 0.1" rpy="0 0 0"/>
-    </xacro:sensor_d435>
+    </xacro:sensor_d435> -->
     <!-- IMU sensor -->
     <joint name="imu_joint" type="fixed">
-        <axis xyz="1 0 0"/> <!-- 0 1 0 -->
-        <origin xyz="-0.05 0 0.14"/>
-        <parent link="base_link"/>
-        <child link="imu_link"/>
+        <axis xyz="1 0 0" /> <!-- 0 1 0 -->
+        <origin xyz="-0.05 0 0.14" />
+        <parent link="base_link" />
+        <child link="imu_link" />
     </joint>
     <link name="imu_link">
         <inertial>
-            <mass value="0.001"/>
-            <origin rpy="0 0 0" xyz="0 0 0"/>
-            <inertia ixx="0.0001" ixy="0" ixz="0" iyy="0.000001" iyz="0" izz="0.0001"/>
+            <mass value="0.001" />
+            <origin rpy="0 0 0" xyz="0 0 0" />
+            <inertia ixx="0.0001" ixy="0" ixz="0" iyy="0.000001" iyz="0" izz="0.0001" />
         </inertial>
         <visual>
-            <origin rpy="0 0 0" xyz="0 0 0"/>
+            <origin rpy="0 0 0" xyz="0 0 0" />
             <geometry>
-                <box size="0.001 0.001 0.001"/>
+                <box size="0.001 0.001 0.001" />
             </geometry>
         </visual>
         <collision>
-            <origin rpy="0 0 0" xyz="0 0 0"/>
+            <origin rpy="0 0 0" xyz="0 0 0" />
             <geometry>
-                <box size=".001 .001 .001"/>
+                <box size=".001 .001 .001" />
             </geometry>
         </collision>
